File: elec_boards/filters/AetS_Spectrum_1way.kicad_pcb (KiCad board)
At the start: 2 copper layers, 86.4 x 52.1 mm, 32 parts, among them J1 Micro_test, J2 Conn_01x06, U1 TL084

Commit message: Update Schematics and PCB
Parts:
- added G***: LOGO, Logos:logo_lense, F.Cu at (236.7, 68.6)
- moved C6 2.53 mm to (175.8, 55.4)
- moved C3 2.46 mm to (175.8, 64.5)
Routing:
- net Vin_micro: track 46.0 -> 49.6 mm
- net VCC+: track 56.2 -> 57.9 mm
- net VCC-: track 46.6 -> 45.4 mm
Other:
- board text added: "Mic_IN"
- board text added: "Nuc_OUT"
- board text added: "OUT"
- board text added: "VCC"
- board text removed: "Nuc_IN"
